File: Hardware/v2/Arturo_Verasv2.brd (EAGLE design)
At the start: 100 x 80 mm, 25 parts, among them T1 BC850, T3 BC850, T4 2SC1815, T5 BC850, T6 BC850, T7 BC850, T8 BC850, X1 22-23-2071, X2 MSTBA12, X3 MSTBA3

Commit message: Más cambios
más cambios en conectores, transistores y resistencias
Parts:
- removed X2: MSTBA12, con-phoenix-508:MSTBA12
- removed X3: MSTBA3, con-phoenix-508:MSTBA3
- added X4: (no value), con-weidmueller-sl35:90F-12
Connections:
- new net N$12: X4.3
- new net N$13: X4.4
- new net N$14: X4.5
- new net N$15: X4.6
- new net N$16: X4.7
- new net N$17: X4.8
- new net N$18: X4.9
- new net N$19: X4.10
- new net N$21: X4.11
- new net N$24: X4.12
- net GENERAL_INPUT+: now also X4.1
- net IGNITION_INPUT+: now also X4.2
Changed lines of the file:
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@@
 <setting verticaltext="up"/>
 </settings>
-<grid distance="50" unitdist="mil" unit="mil" style="lines" multiple="1" display="no" altdistance="5" altunitdist="mil" altunit="mil"/>
+<grid distance="1" unitdist="mil" unit="mil" style="lines" multiple="1" display="no" altdistance="5" altunitdist="mil" altunit="mil"/>
 <layers>
 <layer number="1" name="Top" color="4" fill="1" visible="yes" active="yes"/>
@@
 <attribute name="OC_NEWARK" value="56H0445" x="26.67" y="3.81" size="1.778" layer="27" display="off"/>
 </element>
-<element name="X2" library="con-phoenix-508" library_urn="urn:adsk.eagle:library:176" package="MSTBA12" package3d_urn="urn:adsk.eagle:package:9623/1" value="MSTBA12" x="31.75" y="6.35">
-<attribute name="MF" value="" x="31.75" y="6.35" size="1.778" layer="27" display="off"/>
-<attribute name="MPN" value="1757349" x="31.75" y="6.35" size="1.778" layer="27" display="off"/>
-<attribute name="OC_FARNELL" value="3705250" x="31.75" y="6.35" size="1.778" layer="27" display="off"/>
-<attribute name="OC_NEWARK" value="71C4169" x="31.75" y="6.35" size="1.778" layer="27" display="off"/>
-</element>
-<element name="X3" library="con-phoenix-508" library_urn="urn:adsk.eagle:library:176" package="MSTBA3" package3d_urn="urn:adsk.eagle:package:9608/1" value="MSTBA3" x="7.62" y="-41.91">
-<attribute name="MF" value="FARNELL" x="7.62" y="-41.91" size="1.778" layer="27" display="off"/>
-<attribute name="MPN" value="1757255" x="7.62" y="-41.91" size="1.778" layer="27" display="off"/>
-<attribute name="OC_FARNELL" value="3705183" x="7.62" y="-41.91" size="1.778" layer="27" display="off"/>
-<attribute name="OC_NEWARK" value="71C4162" x="7.62" y="-41.91" size="1.778" layer="27" display="off"/>
+<element name="X4" library="con-weidmueller-sl35" library_urn="urn:adsk.eagle:library:199" package="90F-12" package3d_urn="urn:adsk.eagle:package:11421/1" value="" x="61.5188" y="13.2588">
+<attribute name="MF" value="" x="61.5188" y="13.2588" size="1.778" layer="27" display="off"/>
+<attribute name="MPN" value="" x="61.5188" y="13.2588" size="1.778" layer="27" display="off"/>
+<attribute name="OC_FARNELL" value="unknown" x="61.5188" y="13.2588" size="1.778" layer="27" display="off"/>
+<attribute name="OC_NEWARK" value="unknown" x="61.5188" y="13.2588" size="1.778" layer="27" display="off"/>
 </element>
 </elements>
@@
 <contactref element="R8" pad="2"/>
 <contactref element="X1" pad="2"/>
+<contactref element="X4" pad="2"/>
+<wire x1="26.67" y1="14.29" x2="45.7688" y2="18.5088" width="0" layer="19" extent="1-1"/>
 <wire x1="21.59" y1="3.81" x2="26.67" y2="14.29" width="0" layer="19" extent="1-1"/>
 </signal>
@@
 <contactref element="R12" pad="2"/>
 <contactref element="X1" pad="7"/>
-<wire x1="34.29" y1="3.81" x2="33.02" y2="54.93" width="0" layer="19" extent="1-1"/>
+<contactref element="X4" pad="1"/>
+<wire x1="42.2688" y1="18.5088" x2="33.02" y2="54.93" width="0" layer="19" extent="1-1"/>
+<wire x1="34.29" y1="3.81" x2="42.2688" y2="18.5088" width="0" layer="19" extent="1-1"/>
 </signal>
 <signal name="DGENERAL_INPUT">
@@
 <wire x1="24.13" y1="3.81" x2="26.67" y2="39.37" width="0" layer="19" extent="1-1"/>
 </signal>
+<signal name="N$12">
+<contactref element="X4" pad="3"/>
+</signal>
+<signal name="N$13">
+<contactref element="X4" pad="4"/>
+</signal>
+<signal name="N$14">
+<contactref element="X4" pad="5"/>
+</signal>
+<signal name="N$15">
+<contactref element="X4" pad="6"/>
+</signal>
+<signal name="N$16">
+<contactref element="X4" pad="7"/>
+</signal>
+<signal name="N$17">
+<contactref element="X4" pad="8"/>
+</signal>
+<signal name="N$18">
+<contactref element="X4" pad="9"/>
+</signal>
+<signal name="N$19">
+<contactref element="X4" pad="10"/>
+</signal>
+<signal name="N$21">
+<contactref element="X4" pad="11"/>
+</signal>
+<signal name="N$24">
+<contactref element="X4" pad="12"/>
+</signal>
 </signals>
